File: DeerMon.kicad_pcb (KiCad board)
At the start: 2 copper layers, 30 x 30 mm, 41 parts, among them J1 TYPE-C-31-M-12, J2 ZJY144S025, J3 GPIO, Q1 BC847BVC-7, Q2 2N7002, SW1 BOOT, SW2 EN, U1 CP2102N-A02-GQFN24R, U2 AW9364DNR, U3 SPX3819M5-L-3-3, U4 ESP32-PICO-V3-02

Commit message: Convert to 4 layers PCB
Other:
- copper layers 2 -> 4
Changed lines of the file:
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@@
 (kicad_pcb (version 20171130) (host pcbnew "(5.1.12-1-10_14)")
   (general
-    (thickness 1.2)
+    (thickness 1.4)
     (drawings 11)
     (tracks 315)
@@
   (layers
     (0 F.Cu signal)
+    (1 GND.Cu power)
+    (2 PWR.Cu power)
     (31 B.Cu signal)
     (32 B.Adhes user)

Commit message: Update PCB layout
Parts:
- removed R11: 0, Resistor_SMD:R_0402_1005Metric
- removed TP1: IO5, TestPoint:TestPoint_Pad_D1.0mm
- moved Q1 9.76 mm to (62.6, 68.3), turned to 225 degrees
- moved R1 1.24 mm to (71.1, 61.9)
- moved C1 1.01 mm to (72.3, 65.0)
- moved C2 1.01 mm to (71.6, 65.8)
- moved R2 0.74 mm to (71.8, 62.6)
- moved R5 0.25 mm to (70.4, 61.2)
Connections:
- C1 pad 1: Net-(C1-Pad1) -> +3V3
- C2 pad 1: Net-(C1-Pad1) -> +3V3
- R5 pad 2: Net-(C1-Pad1) -> +3V3
- U1 pad 5: Net-(C1-Pad1) -> +3V3
- U1 pad 6: Net-(C1-Pad1) -> +3V3
- U1 pad 7: Net-(C1-Pad1) -> +3V3
Routing:
- net +3V3: track 31.5 -> 67.2 mm, vias 3 -> 7
- net /EN: track 5.65 -> 30.9 mm, vias 0 -> 1
- net /BOOT: track 35.9 -> 53.3 mm, vias 2 -> 3
- net +5V: track 42.3 -> 59.4 mm
- net /ESP_RX: track 20.0 -> 28.2 mm
- net /ESP_TX: track 18.4 -> 26.3 mm
- net Net-(Q1-Pad1): track 0.00 -> 4.81 mm
- net Net-(Q1-Pad2): track 0.00 -> 4.15 mm
- net Net-(C4-Pad1): track 0.00 -> 1.32 mm
- net GND: vias 13 -> 22
- added copper zone on F.Cu, net +3V3
- added copper zone on GND.Cu, net GND
- added copper zone on PWR.Cu, net GND
Other:
- board text removed: "IO5"

Commit message: Redraw power
Parts:
- added C14: 1uF, Capacitor_SMD:C_0402_1005Metric, F.Cu at (59.9, 69.8)
- added C15: 1uF, Capacitor_SMD:C_0402_1005Metric, F.Cu at (54.4, 70.0)
- added C16: 0.1uF, Capacitor_SMD:C_0402_1005Metric, F.Cu at (55.0, 70.7)
- added C5: 0.1uF, Capacitor_SMD:C_0402_1005Metric, F.Cu at (51.0, 61.9)
- added C6: 10uF, Capacitor_SMD:C_0402_1005Metric, F.Cu at (60.6, 70.5)
- added C7: 100pF, Capacitor_SMD:C_0402_1005Metric, F.Cu at (53.7, 69.3)
- added D4: SK6805-EC15, JLC-SMT:LED_SK6805_EC15_1.5x1.5mm, F.Cu at (58.2, 75.0)
- added R11: 10K, Resistor_SMD:R_0402_1005Metric, F.Cu at (58.2, 73.5)
- C12: value 10uF/6.3V -> 0.1uF
- C13, C2: value 100nF -> 0.1uF
- moved C12 9.17 mm to (59.5, 60.3), turned to 45 degrees
- moved R10 2.00 mm to (58.6, 68.5), turned to 225 degrees
- moved C11 0.83 mm to (60.6, 67.8), turned to 225 degrees
- moved C13 0.28 mm to (59.2, 69.2), turned to 225 degrees
- moved Q1 0.25 mm to (62.6, 68.0)
- moved R12 0.21 mm to (59.9, 67.1)
- moved R9 0.15 mm to (66.3, 67.3)
- moved R8 0.11 mm to (65.7, 66.6)
- moved C1 0.08 mm to (72.2, 65.1)
- moved R7 0.08 mm to (65.0, 65.9)
- moved R2 0.08 mm to (71.7, 62.6)
- moved R5 0.06 mm to (70.4, 61.2)
- moved R1 0.06 mm to (71.0, 61.9)
Connections:
- C12 pad 1: /ESP_VDD -> +3V3
- C13 pad 1: /ESP_VDD -> +3V3
- J3 pad 10: /ESP_RX -> /IO5
- J3 pad 2: +5V -> +3V3
- J3 pad 3: (no net) -> GND
- J3 pad 4: +3V3 -> +5V
- J3 pad 5: (no net) -> /ESP_RX
- J3 pad 6: (no net) -> /ESP_TX
- J3 pad 7: /ESP_TX -> /IO19
- J3 pad 8: (no net) -> /IO22
- R10 pad 1: /ESP_VDD -> +3V3
- R10 pad 2: +3V3 -> Net-(R10-Pad2)
- R12 pad 1: /ESP_VDD -> +3V3
- U4 pad 1: /ESP_VDD -> +3V3
- U4 pad 19: /ESP_VDD -> +3V3
- U4 pad 3: /ESP_VDD -> Net-(R10-Pad2)
- U4 pad 37: /ESP_VDD -> +3V3
- U4 pad 4: /ESP_VDD -> Net-(R10-Pad2)
- U4 pad 42: /IO21 -> /RMT_RGB
- U4 pad 43: /ESP_VDD -> +3V3
- U4 pad 46: /ESP_VDD -> +3V3
Routing:
- net +3V3: track 67.2 -> 121.2 mm, vias 7 -> 11
- net /IO22: track 2.23 -> 34.7 mm
- net /IO19: track 6.04 -> 36.4 mm
- net /IO5: track 2.50 -> 30.4 mm, vias 0 -> 1
- net /ESP_VDD: track 26.1 -> 0.00 mm, vias 6 -> 0
- net /RMT_RGB: track 0.00 -> 13.8 mm, vias 0 -> 2
- net /ESP_RX: track 28.2 -> 41.8 mm
- net /ESP_TX: track 26.3 -> 36.5 mm
- net +5V: track 59.4 -> 52.5 mm
- net /D+: track 18.0 -> 21.2 mm
- net /IO21: track 2.77 -> 0.00 mm, vias 1 -> 0
- net /D-: track 19.6 -> 22.2 mm
- net /BOOT: track 53.3 -> 55.0 mm
- net /LCD_SDA: track 13.2 -> 14.1 mm
- net GND: track 3.44 -> 3.40 mm, vias 22 -> 66
- added copper zone on F.Cu, net Net-(R10-Pad2)
- removed copper zone on F.Cu, net /ESP_VDD

Commit message: Finish PCB
Parts:
- moved C10 1.00 mm to (71.5, 70.0)
- moved C4 1.00 mm to (73.5, 70.6)
- moved C9 1.00 mm to (72.5, 77.8)
- moved R14 1.00 mm to (72.5, 76.2)
- moved U3 1.00 mm to (72.5, 73.5)
- moved AE1 0.56 mm to (52.0, 76.0)
Routing:
- net +3V3: track 121.2 -> 118.8 mm
- net GND: vias 66 -> 108
- added copper zone on F.Cu, net Net-(AE1-Pad1)
Other:
- outline, holes or cut-outs redrawn

Commit message: Update BOM and documents
Parts:
- BZ1: value TMB12A05 -> HMB1206-05; footprint Buzzer_Beeper:Buzzer_12x9.5RM7.6 -> JLC-SMT:HNDZ_TMB1206-05
Changed lines of the file:
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@@
     (diff_pair_gap 0.15)
+  )
+  (module JLC-SMT:HNDZ_TMB1206-05 locked (layer B.Cu)
+    (at 64.8 61.9 135)
+    (descr "Buzzer, D12mm height 6.5mm with RM7.6mm")
+    (tags buzzer)
+    (fp_text reference BZ1 (at 3.8 7.2 135) (layer B.Fab)
+      (effects (font (size 1 1) (thickness 0.15)) (justify mirror))
+    )
+    (fp_text value HMB1206-05 (at 3.8 -7.4 135) (layer B.Fab)
+      (effects (font (size 1 1) (thickness 0.15)) (justify mirror))
+    )
+    (fp_circle (center 3.8 0) (end 10.05 0) (layer B.CrtYd) (width 0.05))
+    (fp_circle (center 3.8 0) (end 9.8 0) (layer B.Fab) (width 0.1))
+    (fp_circle (center 3.8 0) (end 4.8 0) (layer B.Fab) (width 0.1))
+    (fp_circle (center 3.8 0) (end 9.9 0) (layer B.SilkS) (width 0.12))
+    (fp_text user %R (at 3.8 4 135) (layer B.Fab)
+      (effects (font (size 1 1) (thickness 0.15)) (justify mirror))
+    )
+    (fp_text user + (at -0.01 2.54 135) (layer B.SilkS)
+      (effects (font (size 1 1) (thickness 0.15)) (justify mirror))
+    )
+    (fp_text user + (at -0.01 2.54 135) (layer B.Fab)
+      (effects (font (size 1 1) (thickness 0.15)) (justify mirror))
+    )
+    (pad 2 thru_hole circle (at 7.6 0 135) (size 2 2) (drill 1) (layers *.Cu *.Mask)
+      (net 34 "Net-(BZ1-Pad2)"))
+    (pad 1 thru_hole circle (at 0 0 135) (size 2 2) (drill 1) (layers *.Cu *.Mask)
+      (net 5 +5V))
+    (model ${CUSTOM_DIR}/HNDZ_HMB1206-05.step
+      (offset (xyz 3.75 0 0))
+      (scale (xyz 1 1 1))
+      (rotate (xyz 0 0 180))
+    )
   )
   (module Capacitor_SMD:C_0402_1005Metric (layer F.Cu)
@@
       (scale (xyz 1 1 1))
       (rotate (xyz 0 0 0))
-    )
-  )
-  (module Buzzer_Beeper:Buzzer_12x9.5RM7.6 locked (layer B.Cu)
-    (at 64.8 61.9 135)
-    (descr "Generic Buzzer, D12mm height 9.5mm with RM7.6mm")
-    (tags buzzer)
-    (fp_text reference BZ1 (at 3.8 7.2 135) (layer B.Fab)
-      (effects (font (size 1 1) (thickness 0.15)) (justify mirror))
-    )
-    (fp_text value TMB12A05 (at 3.8 -7.4 135) (layer B.Fab)
-      (effects (font (size 1 1) (thickness 0.15)) (justify mirror))
-    )
-    (fp_circle (center 3.8 0) (end 9.9 0) (layer B.SilkS) (width 0.12))
-    (fp_circle (center 3.8 0) (end 4.8 0) (layer B.Fab) (width 0.1))
-    (fp_circle (center 3.8 0) (end 9.8 0) (layer B.Fab) (width 0.1))
-    (fp_circle (center 3.8 0) (end 10.05 0) (layer B.CrtYd) (width 0.05))
-    (fp_text user %R (at 3.8 4 135) (layer B.Fab)
-      (effects (font (size 1 1) (thickness 0.15)) (justify mirror))
-    )
-    (fp_text user + (at -0.01 2.54 135) (layer B.SilkS)
-      (effects (font (size 1 1) (thickness 0.15)) (justify mirror))
-    )
-    (fp_text user + (at -0.01 2.54 135) (layer B.Fab)
-      (effects (font (size 1 1) (thickness 0.15)) (justify mirror))
-    )
-    (pad 2 thru_hole circle (at 7.6 0 135) (size 2 2) (drill 1) (layers *.Cu *.Mask)
-      (net 34 "Net-(BZ1-Pad2)"))
-    (pad 1 thru_hole rect (at 0 0 135) (size 2 2) (drill 1) (layers *.Cu *.Mask)
-      (net 5 +5V))
-    (model ${KISYS3DMOD}/Buzzer_Beeper.3dshapes/Buzzer_12x9.5RM7.6.wrl
-      (at (xyz 0 0 0))
-      (scale (xyz 1 1 1))
-      (rotate (xyz 0 0 0))

Commit message: Finish silk screen
Other:
- board text added: "BOOT 26 33 35 5 22 TX 5V 3V3"
- board text added: "DeerMon"
- board text added: "EN 27 25 32 34 19 RX G G"
- board text added: "V1.0 by XiNGRZ"
Changed lines of the file:
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@@
   (general
     (thickness 1.4)
-    (drawings 18)
+    (drawings 22)
     (tracks 565)
     (zones 0)
@@
     )
   )
+  (gr_text "BOOT\n\n26\n\n33\n\n35\n\n5\n\n22\n\nTX\n\n5V\n\n3V3" (at 72.5 68.05) (layer B.SilkS)
+    (effects (font (size 0.77 0.7) (thickness 0.12)) (justify left mirror))
+  )
+  (gr_text "EN\n\n27\n\n25\n\n32\n\n34\n\n19\n\nRX\n\nG\n\nG" (at 74.2 68.05) (layer B.SilkS)
+    (effects (font (size 0.77 0.7) (thickness 0.12)) (justify left mirror))
+  )
+  (gr_text "V1.0 by XiNGRZ" (at 61.75 59.5) (layer F.SilkS)
+    (effects (font (size 0.8 0.8) (thickness 0.12)) (justify left))
+  )
+  (gr_text DeerMon (at 61.5 57.75) (layer F.SilkS)
+    (effects (font (size 1.2 1.2) (thickness 0.2)) (justify left))
+  )
   (gr_line (start 79.7 79.5) (end 79.7 50.5) (layer Margin) (width 0.15))
